File: AnthC-M1R1/Power.sch (KiCad schematic (older format))
At the start: 30 parts, among them Q8 SI2347DS-T1-GE3, Q9 SI2347DS-T1-GE3, U1 TPS54331DR, U3 TPS78533

Commit message: Assigned some footprints
Added more libraries
Parts:
- D14, D24: footprint (none) -> Semiconductors:D_SOD-123
- U3: footprint (none) -> IC:HVSON-8-1EP_3x3mm_P0.65mm_EP1.6x2.4mm
Changed lines of the file:
@@
 F 0 "U3" H 8700 2515 50  0000 C CNN
 F 1 "TPS78533" H 8700 2424 50  0000 C CNN
-F 2 "" H 8500 1950 50  0001 C CNN
+F 2 "IC:HVSON-8-1EP_3x3mm_P0.65mm_EP1.6x2.4mm" H 8500 1950 50  0001 C CNN
 F 3 "https://www.ti.com/lit/ds/symlink/tps785-q1.pdf" H 8500 1950 50  0001 C CNN
 F 4 "Texas Instruments" H 9650 2600 50  0001 C CNN "Manufacturer"
@@
 F 0 "D14" V 1650 1680 50  0000 L CNN
 F 1 "Zener_6V" V 1695 1680 50  0001 L CNN
-F 2 "" H 1650 1425 50  0001 C CNN
+F 2 "Semiconductors:D_SOD-123" H 1650 1425 50  0001 C CNN
 F 3 "https://www.mouser.be/datasheet/2/427/VISH_S_A0003941535_1-2569124.pdf" H 1650 1600 50  0001 C CNN
 F 4 "Vishay" H 1950 2200 50  0001 C CNN "Manufacturer"
@@
 F 0 "D24" V 7200 1830 50  0000 L CNN
 F 1 "Zener_6V" V 7245 1830 50  0001 L CNN
-F 2 "" H 7200 1575 50  0001 C CNN
+F 2 "Semiconductors:D_SOD-123" H 7200 1575 50  0001 C CNN
 F 3 "https://www.mouser.be/datasheet/2/427/VISH_S_A0003941535_1-2569124.pdf" H 7200 1750 50  0001 C CNN
 F 4 "Vishay" H 7500 2350 50  0001 C CNN "Manufacturer"
