File: AnthC-M1R1/Power.sch (KiCad schematic (older format))
At the start: 30 parts, among them Q8 SI2347DS-T1-GE3, Q9 SI2347DS-T1-GE3, U1 TPS54331DR, U3 TPS78533

Commit message: Added STEP model and a PDF with the top an bottom views
Board ready for manufacturing and assembly
Parts:
- removed D19: B5819W, Diode_SMD:D_SOD-123, symbol AnthC-Lib-Symbols:1N5820
- removed U3: TPS78533, IC:HVSON-8-1EP_3x3mm_P0.65mm_EP1.6x2.4mm, symbol DCDC:TPS78533
- added U3: BD33FC0FP-E2, IC:TO-252-2, symbol DCDC:BD33FC0FP-E2
- R2: footprint Resistor_SMD:R_0603_1608Metric -> Resistor_SMD:R_0201_0603Metric_Pad0.64x0.40mm_HandSolder; symbol Resistor_0603:49.9 -> Resistor_0201:49.9; Description 33 kOhms ±1% 0.1W, 1/10W Chip Resistor 0603 (1608 Metric) M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 -> Resistor Thin Film 49.9Ohm 0.1% 2-Pin 0201 Paper T/R; Manufacturer Nr. TNPW020149R9BEED -> (none)
Connections:
- net 5VD is gone; now on net +5VD: Q9.3 (D)
- net +3V3: now also U3.3 (Vout)
- net +5V: now also U3.1 (Vin)
- net GND: now also U3.2 (GND)
- net +5VD: now reaches C10.1, C11.1, C9.1, L1.2, R8.2
Other:
- moved on the sheet: C22, C24, R86
